File: i2s-shifter.sch (EAGLE design)
At the start: 22 parts, among them IC1 74HC164D, IC2 74HC164D, IC3 74HC164D, IC4 74HC164D, IC5 74HC164D

Commit message: moved caps closer to vcc
Connections:
- net GND renamed NS999
Changed lines of the file:
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@@
 </busses>
 <nets>
-<net name="GND" class="0">
+<net name="NS999" class="0">
 <segment>
 <pinref part="IC1" gate="P" pin="GND"/>
