File: dac_rev0.brd (EAGLE design)
At the start: 99.1 x 49.5 mm, 85 parts, among them IC1 PCM1794A, IC2 PCM1794A

Commit message: minor tweak
Routing:
- net N$23: track 13.7 -> 15.4 mm
- net N$2: track 7.84 -> 8.49 mm
Changed lines of the file:
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@@
 <contactref element="DATA" pad="MP"/>
 <contactref element="R2" pad="1"/>
-<wire x1="22.86" y1="31.75" x2="18.7325" y2="34.6075" width="0.4064" layer="1"/>
+<wire x1="18.7325" y1="34.6075" x2="20.32" y2="33.02" width="0.4064" layer="1"/>
+<wire x1="20.32" y1="33.02" x2="21.9075" y2="33.02" width="0.4064" layer="1"/>
+<wire x1="21.9075" y1="33.02" x2="22.86" y2="32.0675" width="0.4064" layer="1"/>
+<wire x1="22.86" y1="32.0675" x2="22.86" y2="31.75" width="0.4064" layer="1"/>
 </signal>
 <signal name="N$4">
@@
 <contactref element="R1" pad="1"/>
 <contactref element="LR" pad="MP"/>
-<wire x1="25.4" y1="31.75" x2="24.4475" y2="34.6075" width="0.4064" layer="1"/>
+<wire x1="24.4475" y1="34.6075" x2="25.4" y2="33.655" width="0.4064" layer="1"/>
+<wire x1="25.4" y1="33.655" x2="25.4" y2="31.75" width="0.4064" layer="1"/>
 </signal>
 <signal name="N$9">
@@
 <wire x1="13.97" y1="25.4" x2="12.7" y2="25.4" width="0.4064" layer="1"/>
 <wire x1="12.7" y1="25.4" x2="12.7" y2="15.24" width="0.4064" layer="1"/>
-<wire x1="12.7" y1="15.24" x2="16.51" y2="13.97" width="0.4064" layer="1"/>
 <wire x1="28.355" y1="14.155" x2="28.355" y2="16.4125" width="0.4064" layer="1"/>
 <wire x1="28.355" y1="16.4125" x2="28.2575" y2="16.51" width="0.4064" layer="1"/>
@@
 <wire x1="24.13" y1="2.54" x2="62.23" y2="10.16" width="0" layer="19" extent="1-1"/>
 <wire x1="63.5" y1="16.51" x2="28.2575" y2="-40.3225" width="0" layer="19" extent="1-1"/>
+<wire x1="12.7" y1="15.24" x2="13.97" y2="13.97" width="0.4064" layer="1"/>
+<wire x1="13.97" y1="13.97" x2="16.51" y2="13.97" width="0.4064" layer="1"/>
 </signal>
 <signal name="N$14">
@@
 <contactref element="LF80" pad="A1"/>
 <contactref element="L1" pad="2"/>
-<wire x1="33.02" y1="38.1" x2="34.29" y2="36.83" width="1.6764" layer="1"/>
-<wire x1="34.29" y1="36.83" x2="34.925" y2="36.83" width="1.6764" layer="1"/>
-<wire x1="34.925" y1="36.83" x2="40.005" y2="31.75" width="1.6764" layer="1"/>
-<wire x1="40.005" y1="31.75" x2="41.5925" y2="31.75" width="1.6764" layer="1"/>
 <wire x1="38.38" y1="25.14" x2="41.5925" y2="28.3525" width="1.6764" layer="1"/>
 <wire x1="41.5925" y1="28.3525" x2="41.5925" y2="31.75" width="1.6764" layer="1"/>
+<wire x1="33.02" y1="38.1" x2="33.9725" y2="38.1" width="1.6764" layer="1"/>
+<wire x1="33.9725" y1="38.1" x2="40.3225" y2="31.75" width="1.6764" layer="1"/>
+<wire x1="40.3225" y1="31.75" x2="41.5925" y2="31.75" width="1.6764" layer="1"/>
 </signal>
 <signal name="N$23">
@@
 <contactref element="C16" pad="1"/>
 <contactref element="L2" pad="1"/>
-<wire x1="38.38" y1="20.58" x2="35.56" y2="20.32" width="1.27" layer="1"/>
-<wire x1="35.56" y1="20.32" x2="45.72" y2="16.51" width="1.27" layer="1"/>
+<wire x1="35.56" y1="20.32" x2="35.8775" y2="20.6375" width="1.27" layer="1"/>
+<wire x1="35.8775" y1="20.6375" x2="38.4375" y2="20.6375" width="1.27" layer="1"/>
+<wire x1="35.56" y1="20.32" x2="39.37" y2="16.51" width="1.27" layer="1"/>
+<wire x1="39.37" y1="16.51" x2="45.72" y2="16.51" width="1.27" layer="1"/>
+<wire x1="38.38" y1="20.58" x2="38.4375" y2="20.6375" width="1.27" layer="1"/>
+<wire x1="38.4375" y1="20.6375" x2="39.0525" y2="20.6375" width="1.27" layer="1"/>
 </signal>
 <signal name="N$18">
@@
 <contactref element="BCK" pad="MP"/>
 <contactref element="R3" pad="1"/>
-<wire x1="20.32" y1="31.75" x2="13.0175" y2="34.6075" width="0.4064" layer="1"/>
+<wire x1="13.0175" y1="34.6075" x2="15.875" y2="31.75" width="0.4064" layer="1"/>
+<wire x1="15.875" y1="31.75" x2="20.32" y2="31.75" width="0.4064" layer="1"/>
 </signal>
 <signal name="N$8">

Commit message: continue WIP for dac rev0
Parts:
- moved R12 130.2 mm to (83.8, 37.8), turned to 180 degrees
- moved DATA1 125.0 mm to (80.6, 34.9)
- moved BCK1 120.5 mm to (86.4, 34.9)
- moved C32 117.9 mm to (93.3, 35.9), turned to 180 degrees
- moved LR1 108.8 mm to (74.9, 35.2)
- moved DGND1 105.5 mm to (77.8, 34.9)
- moved BGND1 104.6 mm to (83.5, 34.9)
- moved COM1 103.8 mm to (89.9, 2.22)
- moved C34 100.9 mm to (94.6, 16.8)
- moved C26 97.4 mm to (78.4, 11.7), turned to 180 degrees
- moved LGND1 95.3 mm to (72.1, 35.2)
- moved R4 92.0 mm to (72.1, 30.2), turned to 270 degrees
- moved C33 89.8 mm to (63.5, 22.5), turned to 90 degrees
- moved R8 89.7 mm to (74.6, 30.2), turned to 90 degrees
- moved R9 87.6 mm to (76.8, 30.2), turned to 270 degrees
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